File: Meeprom.sch (KiCad schematic (older format))
At the start: 3 parts, among them J1 Tandy_100_102_200_option_rom, U1 28C256

Commit message: Change license to CC. Add Meeprom. Add copper pours.
Parts:
- J1: value Tandy_100_102_200_option_rom -> Molex 8878 socket 27C256 pinout; symbol 000_LOCAL:Tandy_100_102_200_option_rom -> 000_LOCAL:27C256
Connections:
- net A10: now also J1.21 (A10); no longer J1.2 (A10)
- net A11: now also J1.23 (A11); no longer J1.20 (A11)
- net A12: now also J1.2 (A12); no longer J1.24 (A12)
- net A13: now also J1.26 (A13); no longer J1.22 (A13)
- net A14: now also J1.27 (A14); no longer J1.28 (A14)
- net A8: now also J1.25 (A8); no longer J1.26 (A8)
- net A9: now also J1.24 (A9); no longer J1.25 (A9)
- net VCC: now also J1.28 (VCC); no longer J1.1 (VCC)
- net ~CE: now also J1.20 (~CE); no longer J1.27 (~CE)
- net ~OE: now also J1.22 (~OE); no longer J1.21 (~OE)
Changed lines of the file:
@@
 D7
 $Comp
-L 000_LOCAL:Tandy_100_102_200_option_rom J1
+L 000_LOCAL:27C256 J1
 U 1 1 5E6792DF
 P 4380 3550
 F 0 "J1" H 4400 4850 50  0000 C CNN
-F 1 "Tandy_100_102_200_option_rom" H 4400 4750 50  0000 C CNN
+F 1 "Molex 8878 socket 27C256 pinout" H 4400 4750 50  0000 C CNN
 F 2 "000_LOCAL:pcb2molex8878" H 4380 3550 50  0001 C CNN
 F 3 "" H 4380 3550 50  0001 C CNN
