File: Meeprom.sch (KiCad schematic (older format))
At the start: 3 parts, among them J1 Molex 8878 socket 27C256 pino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, U1 28C256

Commit message: minor
Parts:
- R1: footprint Resistors_SMD:R_0805 -> 000_LOCAL:R_0805_2012Metric; symbol Device:R_Small -> 000_LOCAL:R
Changed lines of the file:
@@
 	7920 3350 8020 3250
 $Comp
-L Device:R_Small R1
+L 000_LOCAL:R R1
 U 1 1 5D2BF7AB
-P 6650 4930
-F 0 "R1" V 6570 4860 50  0000 C CNN
-F 1 "47k" V 6570 5000 50  0000 C CNN
-F 2 "Resistors_SMD:R_0805" H 6650 4930 50  0001 C CNN
-F 3 "~" H 6650 4930 50  0001 C CNN
-	1    6650 4930
+P 6600 4930
+F 0 "R1" V 6520 4860 50  0000 C CNN
+F 1 "47k" V 6520 5000 50  0000 C CNN
+F 2 "000_LOCAL:R_0805_2012Metric" H 6600 4930 50  0001 C CNN
+F 3 "~" H 6600 4930 50  0001 C CNN
+	1    6600 4930
 	0    1    1    0
 $EndComp
@@
 ~WE
 Wire Wire Line
-	6300 4930 6550 4930
-Wire Wire Line
 	6300 5030 6750 5030
 Wire Wire Line
@@
 Wire Wire Line
 	6300 4250 6790 4250
+Wire Wire Line
+	6300 4930 6450 4930
 Wire Bus Line
 	8020 2550 8020 5240

Commit message: cosmetics
Parts:
- J1: value Molex 8878 socket 27C256 pinout -> Molex 78805 socket 27C256 pinout; footprint 000_LOCAL:pcb2molex8878 -> 000_LOCAL:Molex78805_PCB
- R1: footprint 000_LOCAL:R_0805_2012Metric -> 000_LOCAL:R_0805
Connections:
- net VSS: no longer names the net of U1.14 (VSS)
- net VSS: no longer J1.14 (VSS)
- no-connect marks 0 -> 1
Changed lines of the file:
@@
 U 1 1 5D231C6F
 P 7190 3550
-F 0 "U1" H 7190 4900 50  0000 C CNN
-F 1 "28C256" H 7190 4800 50  0000 C CNN
+F 0 "U1" H 7190 4940 50  0000 C CNN
+F 1 "28C256" H 7190 4860 50  0000 C CNN
 F 2 "000_LOCAL:SOIC-28W" H 7190 3550 50  0001 C CNN
 F 3 "http://ww1.microchip.com/downloads/en/DeviceDoc/doc0006.pdf" H 7190 3550 50  0001 C CNN
@@
 Entry Wire Line
 	6200 2750 6300 2850
-Entry Wire Line
-	6200 2350 6300 2450
-Text Label 6300 2450 0    50   ~ 0
-VCC
 Text Label 6300 2650 0    50   ~ 0
 A0
@@
 Text Label 6300 4450 0    50   ~ 0
 ~CE
-Entry Wire Line
-	6200 4550 6300 4650
-Text Label 6300 4650 0    50   ~ 0
-VSS
 Wire Wire Line
 	7920 2650 7590 2650
@@
 U 1 1 5D2BF7AB
 P 6600 4930
-F 0 "R1" V 6520 4860 50  0000 C CNN
-F 1 "47k" V 6520 5000 50  0000 C CNN
-F 2 "000_LOCAL:R_0805_2012Metric" H 6600 4930 50  0001 C CNN
+F 0 "R1" V 6520 5010 50  0000 C CNN
+F 1 "47k" V 6520 4870 50  0000 C CNN
+F 2 "000_LOCAL:R_0805" H 6600 4930 50  0001 C CNN
 F 3 "~" H 6600 4930 50  0001 C CNN
 	1    6600 4930
-	0    1    1    0
-$EndComp
-Wire Bus Line
-	6200 5240 8020 5240
-Wire Wire Line
-	6300 4650 7190 4650
+	0    -1   1    0
+$EndComp
 Wire Wire Line
 	6300 4450 6790 4450
@@
 Wire Wire Line
 	6300 2650 6790 2650
-Wire Wire Line
-	6300 2450 7190 2450
 Text Label 7920 2650 2    50   ~ 0
 D0
@@
 Entry Wire Line
 	3390 2750 3490 2850
-Entry Wire Line
-	3390 2350 3490 2450
-Text Label 3490 2450 0    50   ~ 0
-VCC
 Text Label 3490 2650 0    50   ~ 0
 A0
@@
 Text Label 3490 4450 0    50   ~ 0
 ~CE
-Entry Wire Line
-	3390 4550 3490 4650
-Text Label 3490 4650 0    50   ~ 0
-VSS
 Wire Wire Line
 	5110 2650 4780 2650
@@
 	3390 5240 5210 5240
 Wire Wire Line
-	3490 4650 4380 4650
-Wire Wire Line
 	3490 4450 3980 4450
 Wire Wire Line
@@
 Wire Wire Line
 	3490 2650 3980 2650
-Wire Wire Line
-	3490 2450 4380 2450
 Text Label 5110 2650 2    50   ~ 0
 D0
@@
 U 1 1 5E6792DF
 P 4380 3550
-F 0 "J1" H 4400 4850 50  0000 C CNN
-F 1 "Molex 8878 socket 27C256 pinout" H 4400 4750 50  0000 C CNN
-F 2 "000_LOCAL:pcb2molex8878" H 4380 3550 50  0001 C CNN
+F 0 "J1" H 4380 4950 50  0000 C CNN
+F 1 "Molex 78805 socket 27C256 pinout" H 4380 4860 50  0000 C CNN
+F 2 "000_LOCAL:Molex78805_PCB" H 4380 3550 50  0001 C CNN
 F 3 "" H 4380 3550 50  0001 C CNN
 	1    4380 3550
 	1    0    0    -1
 $EndComp
+Connection ~ 5210 5240
+Entry Wire Line
+	6200 4830 6300 4930
+Text Label 6300 4930 0    50   ~ 0
+~WE
+Wire Wire Line
+	6300 4250 6790 4250
+Wire Wire Line
+	6300 4930 6450 4930
+NoConn ~ 3980 4250
+$Comp
+L power:VCC #PWR?
+U 1 1 609B2360
+P 7190 2450
+F 0 "#PWR?" H 7190 2300 50  0001 C CNN
+F 1 "VCC" H 7300 2530 50  0000 C CNN
+F 2 "" H 7190 2450 50  0001 C CNN
+F 3 "" H 7190 2450 50  0001 C CNN
+	1    7190 2450
+	1    0    0    -1
+$EndComp
+$Comp
+L power:VCC #PWR?
+U 1 1 609B7237
+P 4380 2450
+F 0 "#PWR?" H 4380 2300 50  0001 C CNN
+F 1 "VCC" H 4490 2530 50  0000 C CNN
+F 2 "" H 4380 2450 50  0001 C CNN
+F 3 "" H 4380 2450 50  0001 C CNN
+	1    4380 2450
+	1    0    0    -1
+$EndComp
+$Comp
+L power:VCC #PWR?
+U 1 1 609B90C2
+P 6750 4930
+F 0 "#PWR?" H 6750 4780 50  0001 C CNN
+F 1 "VCC" V 6750 5130 50  0000 C CNN
+F 2 "" H 6750 4930 50  0001 C CNN
+F 3 "" H 6750 4930 50  0001 C CNN
+	1    6750 4930
+	0    1    1    0
+$EndComp
 Wire Bus Line
 	5210 5240 6200 5240
-Connection ~ 5210 5240
+Wire Bus Line
+	5210 2550 5210 5240
+Wire Bus Line
+	8020 2550 8020 5240
+Wire Bus Line
+	6200 2550 6200 5240
+Wire Bus Line
+	3390 2550 3390 5240
 Connection ~ 6200 5240
-Entry Wire Line
-	6200 4830 6300 4930
-Entry Wire Line
-	6200 4930 6300 5030
-Text Label 6300 4930 0    50   ~ 0
-VCC
-Text Label 6300 5030 0    50   ~ 0
-~WE
-Wire Wire Line
-	6300 5030 6750 5030
-Wire Wire Line
-	6750 5030 6750 4930
-Wire Wire Line
-	6300 4250 6790 4250
-Wire Wire Line
-	6300 4930 6450 4930
-Wire Bus Line
-	8020 2550 8020 5240
-Wire Bus Line
-	5210 2550 5210 5240
-Wire Bus Line
-	3390 2350 3390 5240
-Wire Bus Line
-	6200 2350 6200 5240
+Wire Bus Line
+	6200 5240 8020 5240
 $EndSCHEMATC
