File: Meeprom.sch (KiCad schematic (older format))
At the start: 3 parts, among them J1 Molex 78805 socket 27C256 pin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, U1 28C256

Commit message: update to v004 board outline and carrier
Parts:
- J1: footprint 000_LOCAL:Molex78805_PCB -> 000_LOCAL:Molex78802_PCB_28
Changed lines of the file:
@@
 Sheet 1 1
 Title "28C256 EEPROM to Molex 78805 socket with 27C256 pinout"
-Date "2021-05-20"
-Rev ""
+Date "2021-05-22"
+Rev "004"
 Comp ""
 Comment1 ""
@@
 F 0 "J1" H 4380 4950 50  0000 C CNN
 F 1 "Molex 78805 socket 27C256 pinout" H 4380 4860 50  0000 C CNN
-F 2 "000_LOCAL:Molex78805_PCB" H 4380 3550 50  0001 C CNN
+F 2 "000_LOCAL:Molex78802_PCB_28" H 4380 3550 50  0001 C CNN
 F 3 "" H 4380 3550 50  0001 C CNN
 	1    4380 3550
