File: FlashOpt100_programming_adapter.sch (KiCad schematic (older format))
At the start: 2 parts, among them J1 29F256, J2 29F256

Commit message: completely new FlashOpt100 and programming adapter
Parts:
- J1: value 29F256 -> 29F256 / 29C256
- J2: value 29F256 -> FlashOpt100_PRG_4x7; footprint 000_LOCAL:4x7_prg_2.0mm_male_straight -> 000_LOCAL:FlashOpt100_PRG_4x7_male; symbol 000_LOCAL:29C256 -> 000_LOCAL:FlashOpt100_PRG_4x7
Connections:
- net A0: now also J2.16 (Pin_16); no longer J2.10 (A0)
- net A1: now also J2.15 (Pin_15); no longer J2.9 (A1)
- net A10: now also J2.27 (Pin_27); no longer J2.21 (A10)
- net A11: now also J2.1 (Pin_1); no longer J2.23 (A11)
- net A12: now also J2.8 (Pin_8); no longer J2.2 (A12)
- net A13: now also J2.4 (Pin_4); no longer J2.26 (A13)
- net A14: now also J2.5 (Pin_5); no longer J2.27 (A14)
- net A2: now also J2.14 (Pin_14); no longer J2.8 (A2)
- net A3: now also J2.13 (Pin_13); no longer J2.7 (A3)
- net A4: now also J2.12 (Pin_12); no longer J2.6 (A4)
- net A5: now also J2.11 (Pin_11); no longer J2.5 (A5)
- net A6: now also J2.10 (Pin_10); no longer J2.4 (A6)
- net A7: now also J2.9 (Pin_9); no longer J2.3 (A7)
- net A8: now also J2.3 (Pin_3); no longer J2.25 (A8)
- net A9: now also J2.2 (Pin_2); no longer J2.24 (A9)
- net D0: now also J2.17 (Pin_17); no longer J2.11 (D0)
- net D1: now also J2.18 (Pin_18); no longer J2.12 (D1)
- net D2: now also J2.19 (Pin_19); no longer J2.13 (D2)
- net D3: now also J2.21 (Pin_21); no longer J2.15 (D3)
- net D4: now also J2.22 (Pin_22); no longer J2.16 (D4)
- net D5: now also J2.23 (Pin_23); no longer J2.17 (D5)
- net D6: now also J2.24 (Pin_24); no longer J2.18 (D6)
- net D7: now also J2.25 (Pin_25); no longer J2.19 (D7)
- net GND: now also J2.20 (Pin_20); no longer J2.14 (GND)
- net VCC: now also J2.7 (Pin_7); no longer J2.28 (VCC)
- net ~CE: now also J2.26 (Pin_26); no longer J2.20 (~CE)
- net ~OE: now also J2.28 (Pin_28); no longer J2.22 (~OE)
- net ~WE: now also J2.6 (Pin_6); no longer J2.1 (~WE)
Other:
- note added: "DIP28 pins to programmer.\n29F256/29C256 DIP28 pinout."
- note added: "For TL-866 programmer, specify device "AT29C256@DIP28" and override chip id mismatch."
- note added: "custom pinout to FlashOpt100"
- note removed: "Pins to programmer ZIF socket."
- note removed: "Programming Port\n29F256/29C256 pinout\nin custom pin header"
- moved on the sheet: J2
Changed lines of the file:
@@
 $EndDescr
 $Comp
-L 000_LOCAL:29C256 J2
+L 000_LOCAL:FlashOpt100_PRG_4x7 J2
 U 1 1 5FAC773B
-P 6870 4000
-F 0 "J2" H 6870 5250 50  0000 C CNN
-F 1 "29F256" H 6870 5340 50  0000 C CNN
-F 2 "000_LOCAL:4x7_prg_2.0mm_male_straight" H 6870 4000 50  0001 C CNN
-F 3 "http://ww1.microchip.com/downloads/en/DeviceDoc/doc0014.pdf" H 6870 4000 50  0001 C CNN
-	1    6870 4000
+P 6500 3700
+F 0 "J2" H 6550 4590 50  0000 C CNN
+F 1 "FlashOpt100_PRG_4x7" H 6550 4700 50  0000 C CNN
+F 2 "000_LOCAL:FlashOpt100_PRG_4x7_male" H 6500 3700 50  0001 C CNN
+F 3 "http://ww1.microchip.com/downloads/en/DeviceDoc/doc0014.pdf" H 6500 3700 50  0001 C CNN
+	1    6500 3700
 	1    0    0    -1
 $EndComp
@@
 	6000 4300 6100 4400
 Entry Wire Line
-	6000 4400 6100 4500
-Entry Wire Line
 	6000 3900 6100 4000
 Entry Wire Line
@@
 	6000 4100 6100 4200
 Entry Wire Line
-	6000 3600 6100 3700
-Entry Wire Line
 	6000 3700 6100 3800
 Entry Wire Line
@@
 Entry Wire Line
 	6000 3200 6100 3300
-Text Label 6100 3100 0    50   ~ 0
-A0
-Text Label 6100 3200 0    50   ~ 0
-A1
-Text Label 6100 3300 0    50   ~ 0
-A2
-Text Label 6100 3400 0    50   ~ 0
-A3
-Text Label 6100 3500 0    50   ~ 0
-A4
-Text Label 6100 3600 0    50   ~ 0
-A5
-Text Label 6100 3700 0    50   ~ 0
-A6
-Text Label 6100 3800 0    50   ~ 0
-A7
-Text Label 6100 3900 0    50   ~ 0
-A8
-Text Label 6100 4000 0    50   ~ 0
-A9
-Text Label 6100 4100 0    50   ~ 0
-A10
-Text Label 6100 4200 0    50   ~ 0
-A11
-Text Label 6100 4300 0    50   ~ 0
-A12
-Text Label 6100 4400 0    50   ~ 0
-A13
-Text Label 6100 4500 0    50   ~ 0
-A14
-Wire Wire Line
-	6100 4500 6470 4500
-Wire Wire Line
-	6100 4400 6470 4400
-Wire Wire Line
-	6100 4300 6470 4300
-Wire Wire Line
-	6100 4200 6470 4200
-Wire Wire Line
-	6100 4100 6470 4100
-Wire Wire Line
-	6100 4000 6470 4000
-Wire Wire Line
-	6100 3900 6470 3900
-Wire Wire Line
-	6100 3800 6470 3800
-Wire Wire Line
-	6100 3700 6470 3700
-Wire Wire Line
-	6100 3600 6470 3600
-Wire Wire Line
-	6100 3500 6470 3500
-Wire Wire Line
-	6100 3400 6470 3400
-Wire Wire Line
-	6100 3300 6470 3300
-Wire Wire Line
-	6100 3200 6470 3200
-Wire Wire Line
-	6100 3100 6470 3100
-Entry Wire Line
-	6000 4600 6100 4700
-Entry Wire Line
-	6000 4800 6100 4900
-Entry Wire Line
-	6000 4700 6100 4800
-Text Label 6100 4900 0    50   ~ 0
-~OE
-Text Label 6100 4800 0    50   ~ 0
-~CE
-Text Label 6100 4700 0    50   ~ 0
-~WE
-Wire Wire Line
-	7600 3100 7270 3100
-Entry Wire Line
-	7600 3100 7700 3000
-Wire Wire Line
-	7600 3200 7270 3200
-Entry Wire Line
-	7600 3200 7700 3100
-Wire Wire Line
-	7600 3300 7270 3300
-Entry Wire Line
-	7600 3300 7700 3200
-Wire Wire Line
-	7600 3400 7270 3400
-Entry Wire Line
-	7600 3400 7700 3300
-Wire Wire Line
-	7600 3500 7270 3500
-Entry Wire Line
-	7600 3500 7700 3400
-Wire Wire Line
-	7600 3600 7270 3600
-Entry Wire Line
-	7600 3600 7700 3500
-Wire Wire Line
-	7600 3700 7270 3700
-Entry Wire Line
-	7600 3700 7700 3600
-Wire Wire Line
-	7600 3800 7270 3800
-Entry Wire Line
-	7600 3800 7700 3700
-Text Label 7600 3100 2    50   ~ 0
-D0
-Text Label 7600 3200 2    50   ~ 0
-D1
-Text Label 7600 3300 2    50   ~ 0
-D2
-Text Label 7600 3400 2    50   ~ 0
-D3
-Text Label 7600 3500 2    50   ~ 0
-D4
-Text Label 7600 3600 2    50   ~ 0
-D5
-Text Label 7600 3700 2    50   ~ 0
-D6
-Text Label 7600 3800 2    50   ~ 0
-D7
-Wire Bus Line
-	6000 5690 7700 5690
-Wire Wire Line
-	6100 4900 6470 4900
-Wire Wire Line
-	6100 4800 6470 4800
-Wire Wire Line
-	6100 4700 6470 4700
-Text Notes 6490 2590 0    50   ~ 0
-Programming Port\n29F256/29C256 pinout\nin custom pin header
+Entry Wire Line
+	7000 3100 7100 3000
+Entry Wire Line
+	7000 3200 7100 3100
+Entry Wire Line
+	7000 3300 7100 3200
+Entry Wire Line
+	7000 3400 7100 3300
+Entry Wire Line
+	7000 3500 7100 3400
+Entry Wire Line
+	7000 3600 7100 3500
+Entry Wire Line
+	7000 3700 7100 3600
+Entry Wire Line
+	7000 3800 7100 3700
+Wire Bus Line
+	6000 5690 7100 5690
+Text Notes 5970 2620 0    50   ~ 0
+custom pinout to FlashOpt100
 $Comp
 L power:GND #PWR0110
 U 1 1 5FB3E48A
-P 6870 5100
-F 0 "#PWR0110" H 6870 4850 50  0001 C CNN
-F 1 "GND" H 6870 4960 50  0000 C CNN
-F 2 "" H 6870 5100 50  0001 C CNN
-F 3 "" H 6870 5100 50  0001 C CNN
-	1    6870 5100
-	1    0    0    -1
+P 6800 3900
+F 0 "#PWR0110" H 6800 3650 50  0001 C CNN
+F 1 "GND" V 6820 3730 50  0000 C CNN
+F 2 "" H 6800 3900 50  0001 C CNN
+F 3 "" H 6800 3900 50  0001 C CNN
+	1    6800 3900
+	0    -1   -1   0
 $EndComp
 $Comp
 L power:VCC #PWR0111
 U 1 1 5FB3F6CB
-P 6870 2900
-F 0 "#PWR0111" H 6870 2750 50  0001 C CNN
-F 1 "VCC" H 6960 2900 50  0000 C CNN
-F 2 "" H 6870 2900 50  0001 C CNN
-F 3 "" H 6870 2900 50  0001 C CNN
-	1    6870 2900
-	1    0    0    -1
+P 6300 3700
+F 0 "#PWR0111" H 6300 3550 50  0001 C CNN
+F 1 "VCC" V 6330 3860 50  0000 C CNN
+F 2 "" H 6300 3700 50  0001 C CNN
+F 3 "" H 6300 3700 50  0001 C CNN
+	1    6300 3700
+	0    -1   -1   0
 $EndComp
 $Comp
@@
 P 3870 4000
 F 0 "J1" H 3870 5250 50  0000 C CNN
-F 1 "29F256" H 3870 5340 50  0000 C CNN
+F 1 "29F256 / 29C256" H 3870 5340 50  0000 C CNN
 F 2 "000_LOCAL:DIP-28_600" H 3870 4000 50  0001 C CNN
 F 3 "http://ww1.microchip.com/downloads/en/DeviceDoc/doc0014.pdf" H 3870 4000 50  0001 C CNN
@@
 Wire Wire Line
 	3100 4700 3470 4700
-Text Notes 3490 2590 0    50   ~ 0
-Pins to programmer ZIF socket.
+Text Notes 3330 2560 0    50   ~ 0
+DIP28 pins to programmer.\n29F256/29C256 DIP28 pinout.
 $Comp
 L power:GND #PWR0101
@@
 Wire Bus Line
 	4700 5690 6000 5690
-Wire Bus Line
-	7700 3000 7700 5690
-Wire Bus Line
-	4700 3000 4700 5690
-Wire Bus Line
-	6000 3000 6000 5690
-Wire Bus Line
-	3000 3000 3000 5690
 Connection ~ 4700 5690
 Connection ~ 6000 5690
+Text Notes 3570 6020 0    50   ~ 0
+For TL-866 programmer, specify device "AT29C256@DIP28" and override chip id mismatch.
+Wire Wire Line
+	6100 3100 6300 3100
+Wire Wire Line
+	6100 3200 6300 3200
+Wire Wire Line
+	6100 3300 6300 3300
+Wire Wire Line
+	6100 3400 6300 3400
+Wire Wire Line
+	6100 3500 6300 3500
+Wire Wire Line
+	6100 3600 6300 3600
+Wire Wire Line
+	6100 3800 6300 3800
+Wire Wire Line
+	6100 3900 6300 3900
+Wire Wire Line
+	6100 4000 6300 4000
+Wire Wire Line
+	6100 4100 6300 4100
+Wire Wire Line
+	6100 4200 6300 4200
+Wire Wire Line
+	6100 4300 6300 4300
+Wire Wire Line
+	6100 4400 6300 4400
+Wire Wire Line
+	6800 3100 7000 3100
+Wire Wire Line
+	6800 3200 7000 3200
+Wire Wire Line
+	6800 3300 7000 3300
+Wire Wire Line
+	6800 3400 7000 3400
+Wire Wire Line
+	6800 3500 7000 3500
+Wire Wire Line
+	6800 3600 7000 3600
+Wire Wire Line
+	6800 3700 7000 3700
+Wire Wire Line
+	6800 3800 7000 3800
+Wire Wire Line
+	6800 4000 7000 4000
+Wire Wire Line
+	6800 4100 7000 4100
+Wire Wire Line
+	6800 4200 7000 4200
+Wire Wire Line
+	6800 4300 7000 4300
+Wire Wire Line
+	6800 4400 7000 4400
+Entry Wire Line
+	7000 4000 7100 3900
+Entry Wire Line
+	7000 4100 7100 4000
+Entry Wire Line
+	7000 4200 7100 4100
+Entry Wire Line
+	7000 4300 7100 4200
+Entry Wire Line
+	7000 4400 7100 4300
+Wire Bus Line
+	4700 3000 4700 5690
+Wire Bus Line
+	6000 3000 6000 5690
+Wire Bus Line
+	3000 3000 3000 5690
+Wire Bus Line
+	7100 3000 7100 5690
+Text Label 6100 3100 0    50   ~ 0
+A11
+Text Label 6100 3200 0    50   ~ 0
+A9
+Text Label 6100 3300 0    50   ~ 0
+A8
+Text Label 6100 3400 0    50   ~ 0
+A13
+Text Label 6100 3500 0    50   ~ 0
+A14
+Text Label 6100 3600 0    50   ~ 0
+~WE
+Text Label 6100 3800 0    50   ~ 0
+A12
+Text Label 6100 3900 0    50   ~ 0
+A7
+Text Label 6100 4000 0    50   ~ 0
+A6
+Text Label 6100 4100 0    50   ~ 0
+A5
+Text Label 6100 4200 0    50   ~ 0
+A4
+Text Label 6100 4300 0    50   ~ 0
+A3
+Text Label 6100 4400 0    50   ~ 0
+A2
+Text Label 7000 4400 2    50   ~ 0
+A1
+Text Label 7000 4300 2    50   ~ 0
+A0
+Text Label 7000 4200 2    50   ~ 0
+D0
+Text Label 7000 4100 2    50   ~ 0
+D1
+Text Label 7000 4000 2    50   ~ 0
+D2
+Text Label 7000 3800 2    50   ~ 0
+D3
+Text Label 7000 3700 2    50   ~ 0
+D4
+Text Label 7000 3600 2    50   ~ 0
+D5
+Text Label 7000 3500 2    50   ~ 0
+D6
+Text Label 7000 3400 2    50   ~ 0
+D7
+Text Label 7000 3300 2    50   ~ 0
+~CE
+Text Label 7000 3200 2    50   ~ 0
+A10
+Text Label 7000 3100 2    50   ~ 0
+~OE
 $EndSCHEMATC
