File: Teeprom.sch (KiCad schematic (older format))
At the start: 3 parts, among them J1 Tandy_100_102_200_option_rom, U1 28C256

Commit message: minor
Parts:
- R1: footprint Resistors_SMD:R_0805 -> 000_LOCAL:R_0805_2012Metric; symbol Device:R_Small -> 000_LOCAL:R
Changed lines of the file:
@@
 	7920 3350 8020 3250
 $Comp
-L Device:R_Small R1
+L 000_LOCAL:R R1
 U 1 1 5D2BF7AB
 P 6650 4930
 F 0 "R1" V 6570 4860 50  0000 C CNN
 F 1 "47k" V 6570 5000 50  0000 C CNN
-F 2 "Resistors_SMD:R_0805" H 6650 4930 50  0001 C CNN
+F 2 "000_LOCAL:R_0805_2012Metric" H 6650 4930 50  0001 C CNN
 F 3 "~" H 6650 4930 50  0001 C CNN
 	1    6650 4930
@@
 ~WE
 Wire Wire Line
-	6300 4930 6550 4930
-Wire Wire Line
-	6300 5030 6750 5030
-Wire Wire Line
-	6750 5030 6750 4930
+	6300 4930 6500 4930
+Wire Wire Line
+	6300 5030 6800 5030
+Wire Wire Line
+	6800 5030 6800 4930
 Wire Wire Line
 	6300 4250 6790 4250

Commit message: cosmetics
Parts:
- J1: footprint 000_LOCAL:pcb2molex8878 -> 000_LOCAL:Molex78805_PCB
- R1: footprint 000_LOCAL:R_0805_2012Metric -> 000_LOCAL:R_0805
Connections:
- net VSS renamed GND
- no-connect marks 0 -> 1
Changed lines of the file:
@@
 Sheet 1 1
 Title "Tandy Model 100/102/200 Option ROM EEPROM"
-Date ""
+Date "2021-05-10"
 Rev ""
 Comp ""
@@
 U 1 1 5D231C6F
 P 7190 3550
-F 0 "U1" H 7190 4900 50  0000 C CNN
-F 1 "28C256" H 7190 4800 50  0000 C CNN
+F 0 "U1" H 7190 5010 50  0000 C CNN
+F 1 "28C256" H 7190 4930 50  0000 C CNN
 F 2 "000_LOCAL:SOIC-28W" H 7190 3550 50  0001 C CNN
 F 3 "http://ww1.microchip.com/downloads/en/DeviceDoc/doc0006.pdf" H 7190 3550 50  0001 C CNN
@@
 Entry Wire Line
 	6200 2750 6300 2850
-Entry Wire Line
-	6200 2350 6300 2450
-Text Label 6300 2450 0    50   ~ 0
-VCC
 Text Label 6300 2650 0    50   ~ 0
 A0
@@
 Text Label 6300 4450 0    50   ~ 0
 ~CE
-Entry Wire Line
-	6200 4550 6300 4650
-Text Label 6300 4650 0    50   ~ 0
-VSS
 Wire Wire Line
 	7920 2650 7590 2650
@@
 U 1 1 5D2BF7AB
 P 6650 4930
-F 0 "R1" V 6570 4860 50  0000 C CNN
-F 1 "47k" V 6570 5000 50  0000 C CNN
-F 2 "000_LOCAL:R_0805_2012Metric" H 6650 4930 50  0001 C CNN
+F 0 "R1" V 6560 5020 50  0000 C CNN
+F 1 "47k" V 6560 4870 50  0000 C CNN
+F 2 "000_LOCAL:R_0805" H 6650 4930 50  0001 C CNN
 F 3 "~" H 6650 4930 50  0001 C CNN
 	1    6650 4930
-	0    1    1    0
-$EndComp
-Wire Bus Line
-	6200 5240 8020 5240
-Wire Wire Line
-	6300 4650 7190 4650
+	0    -1   1    0
+$EndComp
 Wire Wire Line
 	6300 4450 6790 4450
@@
 Wire Wire Line
 	6300 2650 6790 2650
-Wire Wire Line
-	6300 2450 7190 2450
 Text Label 7920 2650 2    50   ~ 0
 D0
@@
 Entry Wire Line
 	3390 2750 3490 2850
-Entry Wire Line
-	3390 2350 3490 2450
-Text Label 3490 2450 0    50   ~ 0
-VCC
 Text Label 3490 2650 0    50   ~ 0
 A0
@@
 Text Label 3490 4450 0    50   ~ 0
 ~CE
-Entry Wire Line
-	3390 4550 3490 4650
-Text Label 3490 4650 0    50   ~ 0
-VSS
 Wire Wire Line
 	5110 2650 4780 2650
@@
 	3390 5240 5210 5240
 Wire Wire Line
-	3490 4650 4380 4650
-Wire Wire Line
 	3490 4450 3980 4450
 Wire Wire Line
@@
 Wire Wire Line
 	3490 2650 3980 2650
-Wire Wire Line
-	3490 2450 4380 2450
 Text Label 5110 2650 2    50   ~ 0
 D0
@@
 U 1 1 5E6792DF
 P 4380 3550
-F 0 "J1" H 4400 4850 50  0000 C CNN
-F 1 "Tandy_100_102_200_option_rom" H 4400 4750 50  0000 C CNN
-F 2 "000_LOCAL:pcb2molex8878" H 4380 3550 50  0001 C CNN
+F 0 "J1" H 4380 4940 50  0000 C CNN
+F 1 "Tandy_100_102_200_option_rom" H 4380 4850 50  0000 C CNN
+F 2 "000_LOCAL:Molex78805_PCB" H 4380 3550 50  0001 C CNN
 F 3 "" H 4380 3550 50  0001 C CNN
 	1    4380 3550
 	1    0    0    -1
 $EndComp
+Connection ~ 5210 5240
+Entry Wire Line
+	6200 4830 6300 4930
+Text Label 6300 4930 0    50   ~ 0
+~WE
+Wire Wire Line
+	6300 4930 6500 4930
+Wire Wire Line
+	6300 4250 6790 4250
+NoConn ~ 3980 4250
+$Comp
+L power:VCC #PWR?
+U 1 1 609B63B2
+P 4380 2450
+F 0 "#PWR?" H 4380 2300 50  0001 C CNN
+F 1 "VCC" H 4480 2530 50  0000 C CNN
+F 2 "" H 4380 2450 50  0001 C CNN
+F 3 "" H 4380 2450 50  0001 C CNN
+	1    4380 2450
+	1    0    0    -1
+$EndComp
+$Comp
+L power:VCC #PWR?
+U 1 1 609B6F25
+P 7190 2450
+F 0 "#PWR?" H 7190 2300 50  0001 C CNN
+F 1 "VCC" H 7290 2530 50  0000 C CNN
+F 2 "" H 7190 2450 50  0001 C CNN
+F 3 "" H 7190 2450 50  0001 C CNN
+	1    7190 2450
+	1    0    0    -1
+$EndComp
+$Comp
+L power:VCC #PWR?
+U 1 1 609B93B5
+P 6800 4930
+F 0 "#PWR?" H 6800 4780 50  0001 C CNN
+F 1 "VCC" V 6800 5120 50  0000 C CNN
+F 2 "" H 6800 4930 50  0001 C CNN
+F 3 "" H 6800 4930 50  0001 C CNN
+	1    6800 4930
+	0    1    1    0
+$EndComp
+$Comp
+L power:GND #PWR?
+U 1 1 609BD5F9
+P 4380 4650
+F 0 "#PWR?" H 4380 4400 50  0001 C CNN
+F 1 "GND" H 4420 4440 50  0000 C CNN
+F 2 "" H 4380 4650 50  0001 C CNN
+F 3 "" H 4380 4650 50  0001 C CNN
+	1    4380 4650
+	1    0    0    -1
+$EndComp
+$Comp
+L power:GND #PWR?
+U 1 1 609BDC96
+P 7190 4650
+F 0 "#PWR?" H 7190 4400 50  0001 C CNN
+F 1 "GND" H 7230 4440 50  0000 C CNN
+F 2 "" H 7190 4650 50  0001 C CNN
+F 3 "" H 7190 4650 50  0001 C CNN
+	1    7190 4650
+	1    0    0    -1
+$EndComp
 Wire Bus Line
 	5210 5240 6200 5240
-Connection ~ 5210 5240
 Connection ~ 6200 5240
-Entry Wire Line
-	6200 4830 6300 4930
-Entry Wire Line
-	6200 4930 6300 5030
-Text Label 6300 4930 0    50   ~ 0
-VCC
-Text Label 6300 5030 0    50   ~ 0
-~WE
-Wire Wire Line
-	6300 4930 6500 4930
-Wire Wire Line
-	6300 5030 6800 5030
-Wire Wire Line
-	6800 5030 6800 4930
-Wire Wire Line
-	6300 4250 6790 4250
+Wire Bus Line
+	6200 5240 8020 5240
 Wire Bus Line
 	8020 2550 8020 5240
@@
 	5210 2550 5210 5240
 Wire Bus Line
-	3390 2350 3390 5240
-Wire Bus Line
-	6200 2350 6200 5240
+	6200 2550 6200 5240
+Wire Bus Line
+	3390 2550 3390 5240
 $EndSCHEMATC

Commit message: update to v004 board outline and carrier
Parts:
- J1: footprint 000_LOCAL:Molex78805_PCB -> 000_LOCAL:Molex78802_PCB_28
Changed lines of the file:
@@
 Sheet 1 1
 Title "Tandy Model 100/102/200 Option ROM EEPROM"
-Date "2021-05-10"
-Rev ""
+Date "2021-05-22"
+Rev "004"
 Comp ""
 Comment1 ""
@@
 F 0 "J1" H 4380 4940 50  0000 C CNN
 F 1 "Tandy_100_102_200_option_rom" H 4380 4850 50  0000 C CNN
-F 2 "000_LOCAL:Molex78805_PCB" H 4380 3550 50  0001 C CNN
+F 2 "000_LOCAL:Molex78802_PCB_28" H 4380 3550 50  0001 C CNN
 F 3 "" H 4380 3550 50  0001 C CNN
 	1    4380 3550
@@
 NoConn ~ 3980 4250
 $Comp
-L power:VCC #PWR?
+L power:VCC #PWR0101
 U 1 1 609B63B2
 P 4380 2450
-F 0 "#PWR?" H 4380 2300 50  0001 C CNN
+F 0 "#PWR0101" H 4380 2300 50  0001 C CNN
 F 1 "VCC" H 4480 2530 50  0000 C CNN
 F 2 "" H 4380 2450 50  0001 C CNN
@@
 $EndComp
 $Comp
-L power:VCC #PWR?
+L power:VCC #PWR0102
 U 1 1 609B6F25
 P 7190 2450
-F 0 "#PWR?" H 7190 2300 50  0001 C CNN
+F 0 "#PWR0102" H 7190 2300 50  0001 C CNN
 F 1 "VCC" H 7290 2530 50  0000 C CNN
 F 2 "" H 7190 2450 50  0001 C CNN
@@
 $EndComp
 $Comp
-L power:VCC #PWR?
+L power:VCC #PWR0103
 U 1 1 609B93B5
 P 6800 4930
-F 0 "#PWR?" H 6800 4780 50  0001 C CNN
+F 0 "#PWR0103" H 6800 4780 50  0001 C CNN
 F 1 "VCC" V 6800 5120 50  0000 C CNN
 F 2 "" H 6800 4930 50  0001 C CNN
@@
 $EndComp
 $Comp
-L power:GND #PWR?
+L power:GND #PWR0104
 U 1 1 609BD5F9
 P 4380 4650
-F 0 "#PWR?" H 4380 4400 50  0001 C CNN
+F 0 "#PWR0104" H 4380 4400 50  0001 C CNN
 F 1 "GND" H 4420 4440 50  0000 C CNN
 F 2 "" H 4380 4650 50  0001 C CNN
@@
 $EndComp
 $Comp
-L power:GND #PWR?
+L power:GND #PWR0105
 U 1 1 609BDC96
 P 7190 4650
-F 0 "#PWR?" H 7190 4400 50  0001 C CNN
+F 0 "#PWR0105" H 7190 4400 50  0001 C CNN
 F 1 "GND" H 7230 4440 50  0000 C CNN
 F 2 "" H 7190 4650 50  0001 C CNN
