File: MEE2732.sch (KiCad schematic (older format))
At the start: 3 parts, among them J1 Molex 78805 socket 27C256 pin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, U1 28C256

Commit message: add MEE2732
Parts:
- added R2, R3: 100k, 000_LOCAL:R_0805, symbol 000_LOCAL:R
- added SW1: SW_SPDT, 000_LOCAL:CL-SB-12C-0x, symbol 000_LOCAL:SW_SPDT
- J1: value Molex 78805 socket 27C256 pinout -> Molex 78805 socket 27C32 pinout; footprint 000_LOCAL:Molex78802_PCB_28 -> 000_LOCAL:Molex78802_PCB_24; symbol 000_LOCAL:27C256 -> 000_LOCAL:27C32
- R1: value 47k -> 100k
- U1: value 28C256 -> 28C64; symbol 000_LOCAL:28C256 -> 000_LOCAL:28C64
Connections:
- net labels removed: A13, A14
- wire segments 52 -> 47
- no-connect marks 1 -> 2
Other:
- moved on the sheet: R1
Changed lines of the file:
@@
 encoding utf-8
 Sheet 1 1
-Title "28C256 EEPROM to Molex 78805 socket with 27C256 pinout"
+Title "28C64 EEPROM to Molex 78805 socket with 2732 pinout"
 Date "2021-05-30"
-Rev "004"
-Comp ""
+Rev "001"
+Comp "b.kenyon.w@gmail.com"
 Comment1 ""
 Comment2 ""
@@
 Comment4 ""
 $EndDescr
-$Comp
-L 000_LOCAL:28C256 U1
-U 1 1 5D231C6F
-P 7190 3550
-F 0 "U1" H 7190 4940 50  0000 C CNN
-F 1 "28C256" H 7190 4860 50  0000 C CNN
-F 2 "000_LOCAL:SOIC-28W" H 7190 3550 50  0001 C CNN
-F 3 "http://ww1.microchip.com/downloads/en/DeviceDoc/doc0006.pdf" H 7190 3550 50  0001 C CNN
-	1    7190 3550
-	1    0    0    -1
-$EndComp
+Entry Wire Line
+	6200 3950 6300 4050
+Entry Wire Line
+	6200 4250 6300 4350
 Entry Wire Line
 	6200 4150 6300 4250
 Entry Wire Line
-	6200 4250 6300 4350
-Entry Wire Line
-	6200 4350 6300 4450
-Entry Wire Line
 	6200 3750 6300 3850
-Entry Wire Line
-	6200 3850 6300 3950
-Entry Wire Line
-	6200 3950 6300 4050
 Entry Wire Line
 	6200 3450 6300 3550
@@
 Text Label 6300 3850 0    50   ~ 0
 A12
-Text Label 6300 3950 0    50   ~ 0
-A13
-Text Label 6300 4050 0    50   ~ 0
-A14
 Text Label 6300 4350 0    50   ~ 0
 ~OE
-Text Label 6300 4450 0    50   ~ 0
+Text Label 6300 4250 0    50   ~ 0
 ~CE
 Wire Wire Line
@@
 L 000_LOCAL:R R1
 U 1 1 5D2BF7AB
-P 6600 4930
-F 0 "R1" V 6520 5010 50  0000 C CNN
-F 1 "47k" V 6520 4870 50  0000 C CNN
-F 2 "000_LOCAL:R_0805" H 6600 4930 50  0001 C CNN
-F 3 "~" H 6600 4930 50  0001 C CNN
-	1    6600 4930
+P 4300 5700
+F 0 "R1" V 4220 5780 50  0000 C CNN
+F 1 "100k" V 4220 5610 50  0000 C CNN
+F 2 "000_LOCAL:R_0805" H 4300 5700 50  0001 C CNN
+F 3 "~" H 4300 5700 50  0001 C CNN
+	1    4300 5700
 	0    -1   1    0
 $EndComp
 Wire Wire Line
-	6300 4450 6790 4450
+	6300 4250 6790 4250
 Wire Wire Line
 	6300 4350 6790 4350
-Wire Wire Line
-	6300 4050 6790 4050
-Wire Wire Line
-	6300 3950 6790 3950
 Wire Wire Line
 	6300 3850 6790 3850
@@
 Text Label 7920 3350 2    50   ~ 0
 D7
-Text Label 6300 4250 0    50   ~ 0
+Text Label 6300 4050 0    50   ~ 0
 ~WE
 Entry Wire Line
 	3390 4250 3490 4350
 Entry Wire Line
-	3390 4350 3490 4450
-Entry Wire Line
-	3390 3750 3490 3850
-Entry Wire Line
-	3390 3850 3490 3950
-Entry Wire Line
-	3390 3950 3490 4050
+	3390 4150 3490 4250
 Entry Wire Line
 	3390 3450 3490 3550
@@
 Text Label 3490 3750 0    50   ~ 0
 A11
-Text Label 3490 3850 0    50   ~ 0
-A12
-Text Label 3490 3950 0    50   ~ 0
-A13
-Text Label 3490 4050 0    50   ~ 0
-A14
 Text Label 3490 4350 0    50   ~ 0
 ~OE
-Text Label 3490 4450 0    50   ~ 0
+Text Label 3490 4250 0    50   ~ 0
 ~CE
 Wire Wire Line
@@
 	5110 3350 5210 3250
 Wire Bus Line
-	3390 5240 5210 5240
-Wire Wire Line
-	3490 4450 3980 4450
+	3390 5240 3700 5240
+Wire Wire Line
+	3490 4250 3980 4250
 Wire Wire Line
 	3490 4350 3980 4350
-Wire Wire Line
-	3490 4050 3980 4050
-Wire Wire Line
-	3490 3950 3980 3950
-Wire Wire Line
-	3490 3850 3980 3850
 Wire Wire Line
 	3490 3750 3980 3750
@@
 Text Label 5110 3350 2    50   ~ 0
 D7
-$Comp
-L 000_LOCAL:27C256 J1
-U 1 1 5E6792DF
-P 4380 3550
-F 0 "J1" H 4380 4950 50  0000 C CNN
-F 1 "Molex 78805 socket 27C256 pinout" H 4380 4860 50  0000 C CNN
-F 2 "000_LOCAL:Molex78802_PCB_28" H 4380 3550 50  0001 C CNN
-F 3 "" H 4380 3550 50  0001 C CNN
-	1    4380 3550
-	1    0    0    -1
-$EndComp
 Connection ~ 5210 5240
 Entry Wire Line
-	6200 4830 6300 4930
-Text Label 6300 4930 0    50   ~ 0
+	3700 5600 3800 5700
+Text Label 3800 5700 0    50   ~ 0
 ~WE
 Wire Wire Line
-	6300 4250 6790 4250
-Wire Wire Line
-	6300 4930 6450 4930
-NoConn ~ 3980 4250
+	6300 4050 6790 4050
+Wire Wire Line
+	3800 5700 4150 5700
 $Comp
 L power:VCC #PWR0101
@@
 L power:VCC #PWR0103
 U 1 1 609B90C2
-P 6750 4930
-F 0 "#PWR0103" H 6750 4780 50  0001 C CNN
-F 1 "VCC" V 6750 5130 50  0000 C CNN
-F 2 "" H 6750 4930 50  0001 C CNN
-F 3 "" H 6750 4930 50  0001 C CNN
-	1    6750 4930
+P 4450 5700
+F 0 "#PWR0103" H 4450 5550 50  0001 C CNN
+F 1 "VCC" V 4450 5900 50  0000 C CNN
+F 2 "" H 4450 5700 50  0001 C CNN
+F 3 "" H 4450 5700 50  0001 C CNN
+	1    4450 5700
 	0    1    1    0
 $EndComp
@@
 Wire Bus Line
 	6200 5240 8020 5240
+$Comp
+L power:GND #PWR0104
+U 1 1 60B44A90
+P 4380 4550
+F 0 "#PWR0104" H 4380 4300 50  0001 C CNN
+F 1 "GND" H 4410 4340 50  0000 C CNN
+F 2 "" H 4380 4550 50  0001 C CNN
+F 3 "" H 4380 4550 50  0001 C CNN
+	1    4380 4550
+	1    0    0    -1
+$EndComp
+$Comp
+L power:GND #PWR0105
+U 1 1 60B47117
+P 7190 4550
+F 0 "#PWR0105" H 7190 4300 50  0001 C CNN
+F 1 "GND" H 7220 4340 50  0000 C CNN
+F 2 "" H 7190 4550 50  0001 C CNN
+F 3 "" H 7190 4550 50  0001 C CNN
+	1    7190 4550
+	1    0    0    -1
+$EndComp
+$Comp
+L 000_LOCAL:R R2
+U 1 1 60B69487
+P 4350 6000
+F 0 "R2" V 4270 6080 50  0000 C CNN
+F 1 "100k" V 4270 5910 50  0000 C CNN
+F 2 "000_LOCAL:R_0805" H 4350 6000 50  0001 C CNN
+F 3 "~" H 4350 6000 50  0001 C CNN
+	1    4350 6000
+	0    -1   1    0
+$EndComp
+Entry Wire Line
+	3700 6000 3800 6100
+Text Label 3800 6100 0    50   ~ 0
+A12
+$Comp
+L power:GND #PWR0106
+U 1 1 60B6FF59
+P 4500 6000
+F 0 "#PWR0106" H 4500 5750 50  0001 C CNN
+F 1 "GND" V 4500 5880 50  0000 R CNN
+F 2 "" H 4500 6000 50  0001 C CNN
+F 3 "" H 4500 6000 50  0001 C CNN
+	1    4500 6000
+	0    -1   -1   0
+$EndComp
+$Comp
+L 000_LOCAL:28C64 U1
+U 1 1 5D231C6F
+P 7190 3450
+F 0 "U1" H 7190 4840 50  0000 C CNN
+F 1 "28C64" H 7190 4760 50  0000 C CNN
+F 2 "000_LOCAL:SOIC-28W" H 7190 3450 50  0001 C CNN
+F 3 "http://ww1.microchip.com/downloads/en/DeviceDoc/doc0006.pdf" H 7190 3450 50  0001 C CNN
+	1    7190 3450
+	1    0    0    -1
+$EndComp
+$Comp
+L 000_LOCAL:27C32 J1
+U 1 1 5E6792DF
+P 4380 3450
+F 0 "J1" H 4380 4850 50  0000 C CNN
+F 1 "Molex 78805 socket 27C32 pinout" H 4380 4760 50  0000 C CNN
+F 2 "000_LOCAL:Molex78802_PCB_24" H 4380 3450 50  0001 C CNN
+F 3 "" H 4380 3450 50  0001 C CNN
+	1    4380 3450
+	1    0    0    -1
+$EndComp
+NoConn ~ 7590 4250
+NoConn ~ 7590 4350
+$Comp
+L 000_LOCAL:R R3
+U 1 1 60BA478F
+P 4350 6200
+F 0 "R3" V 4270 6280 50  0000 C CNN
+F 1 "100k" V 4270 6110 50  0000 C CNN
+F 2 "000_LOCAL:R_0805" H 4350 6200 50  0001 C CNN
+F 3 "~" H 4350 6200 50  0001 C CNN
+	1    4350 6200
+	0    -1   1    0
+$EndComp
+$Comp
+L power:VCC #PWR0107
+U 1 1 60BB5E07
+P 4500 6200
+F 0 "#PWR0107" H 4500 6050 50  0001 C CNN
+F 1 "VCC" V 4500 6400 50  0000 C CNN
+F 2 "" H 4500 6200 50  0001 C CNN
+F 3 "" H 4500 6200 50  0001 C CNN
+	1    4500 6200
+	0    1    1    0
+$EndComp
+Connection ~ 3700 5240
+Wire Bus Line
+	3700 5240 5210 5240
+$Comp
+L 000_LOCAL:SW_SPDT SW1
+U 1 1 60BD570D
+P 4000 6100
+F 0 "SW1" H 4000 6400 50  0000 C CNN
+F 1 "SW_SPDT" H 4000 6300 50  0000 C CNN
+F 2 "000_LOCAL:CL-SB-12C-0x" H 4000 6100 50  0001 C CNN
+F 3 "~" H 4000 6100 50  0001 C CNN
+	1    4000 6100
+	1    0    0    -1
+$EndComp
+Wire Bus Line
+	3700 5240 3700 6000
 Wire Bus Line
 	5210 2550 5210 5240
@@
 Wire Bus Line
 	3390 2550 3390 5240
-$Comp
-L power:GND #PWR0104
-U 1 1 60B3CF4E
-P 4380 4650
-F 0 "#PWR0104" H 4380 4400 50  0001 C CNN
-F 1 "GND" H 4410 4450 50  0000 C CNN
-F 2 "" H 4380 4650 50  0001 C CNN
-F 3 "" H 4380 4650 50  0001 C CNN
-	1    4380 4650
-	1    0    0    -1
-$EndComp
-$Comp
-L power:GND #PWR0105
-U 1 1 60B3D778
-P 7190 4650
-F 0 "#PWR0105" H 7190 4400 50  0001 C CNN
-F 1 "GND" H 7220 4450 50  0000 C CNN
-F 2 "" H 7190 4650 50  0001 C CNN
-F 3 "" H 7190 4650 50  0001 C CNN
-	1    7190 4650
-	1    0    0    -1
-$EndComp
 $EndSCHEMATC
